File: mainboard.brd (EAGLE design)
At the start: 34 x 39.4 mm, 14 parts, among them J1 POWER_JACKPTH, U1 ATMEGA328P

Commit message: Updates
Parts:
- C1, C2: device SparkFun-Capacitors:GRM43D -> SparkFun-Capacitors:0603-CAP
- moved C1 6.84 mm to (19.1, 10.2), turned to 0 degrees
- moved R1 5.68 mm to (11.4, 24.1)
- moved C2 2.54 mm to (15.2, 7.62), turned to 90 degrees
- moved R2 1.27 mm to (5.08, 29.2), turned to 180 degrees
Connections:
- removed net OUT_DISPLAY: JPDISPLAY.1, U1.10
- net DTR: now also C2.1; no longer C2.A
- net GND: now also C1.2, JPDISPLAY.2, JPSPEAKER.1, JPTIMER.1, JPTOGGLE.1; no longer C1.C, JPDISPLAY.3, JPSPEAKER.2, JPTIMER.2, JPTOGGLE.2
- net IN_TIMER: now also JPTIMER.2; no longer JPTIMER.1
- net IN_TOGGLE: now also JPTOGGLE.2; no longer JPTOGGLE.1
- net N$1: now also JPSPEAKER.2; no longer JPSPEAKER.1
- net RESET: now also C2.2; no longer C2.C
- net TX: now also JPDISPLAY.1
- net VCC: now also C1.1, JPDISPLAY.3; no longer C1.A, JPDISPLAY.2
Routing:
- net GND: track 110.2 -> 0.00 mm, vias 1 -> 0
- net RESET: track 71.2 -> 39.7 mm, vias 3 -> 9
- net TX: track 40.5 -> 64.5 mm, vias 1 -> 2
- net OUT_DISPLAY: track 20.1 -> 0.00 mm, vias 1 -> 0
- net RX: track 44.1 -> 24.7 mm, vias 1 -> 7
- net N$1: track 3.07 -> 10.0 mm, vias 0 -> 2
- net VCC: track 88.9 -> 83.7 mm
- net DTR: track 8.93 -> 4.23 mm
- net OUT_SPEAKER: track 6.84 -> 3.92 mm
- net SCK: track 13.6 -> 15.0 mm, vias 1 -> 0
- net MOSI: track 26.6 -> 25.8 mm, vias 1 -> 0
- net MISO: vias 0 -> 3
