File: mainboard.sch (EAGLE design)
At the start: 14 parts, among them J1 POWER_JACKPTH, U1 ATMEGA328P

Commit message: Updates
Parts:
- C1, C2: device SparkFun-Capacitors:CAPSMD -> SparkFun-Capacitors:0.1UF-25V(+80/-20%)(0603)
Connections:
- removed net OUT_DISPLAY: JPDISPLAY.1, U1.PD6(AIN0)
- net GND: now also JPDISPLAY.2, JPSPEAKER.1, JPTIMER.1, JPTOGGLE.1; no longer JPDISPLAY.3, JPSPEAKER.2, JPTIMER.2, JPTOGGLE.2
- net IN_TIMER: now also JPTIMER.2; no longer JPTIMER.1
- net IN_TOGGLE: now also JPTOGGLE.2; no longer JPTOGGLE.1
- net N$1: now also JPSPEAKER.2; no longer JPSPEAKER.1
- net TX: now also JPDISPLAY.1
- net VCC: now also JPDISPLAY.3; no longer JPDISPLAY.2
Other:
- moved on the sheet: R1
Changed lines of the file:
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@@
 <part name="GND7" library="SparkFun-Aesthetics" deviceset="GND" device=""/>
 <part name="J1" library="SparkFun-Connectors" deviceset="POWER_JACK" device="PTH"/>
-<part name="C1" library="SparkFun-Capacitors" deviceset="CAP" device="SMD" value="0.1uF"/>
 <part name="SUPPLY3" library="SparkFun-Aesthetics" deviceset="VCC" device=""/>
 <part name="SUPPLY4" library="SparkFun-Aesthetics" deviceset="VCC" device=""/>
-<part name="C2" library="SparkFun-Capacitors" deviceset="CAP" device="SMD" value="0.1uF"/>
 <part name="GND6" library="SparkFun-Aesthetics" deviceset="GND" device=""/>
 <part name="JAVR" library="SparkFun-Connectors" deviceset="AVR_SPI_PRG_6" device="PTH"/>
@@
 <part name="SUPPLY7" library="SparkFun-Aesthetics" deviceset="VCC" device=""/>
 <part name="JP2" library="SparkFun-Connectors" deviceset="M10" device="LOCK"/>
+<part name="C1" library="SparkFun-Capacitors" deviceset="0.1UF-25V(+80/-20%)(0603)" device="" value="0.1uF"/>
+<part name="C2" library="SparkFun-Capacitors" deviceset="0.1UF-25V(+80/-20%)(0603)" device="" value="0.1uF"/>
 </parts>
 <sheets>
@@
 <instance part="FRAME1" gate="G$1" x="0" y="0"/>
 <instance part="FRAME1" gate="G$2" x="147.32" y="0"/>
-<instance part="R1" gate="G$1" x="106.68" y="124.46"/>
+<instance part="R1" gate="G$1" x="106.68" y="127"/>
 <instance part="U1" gate="G$1" x="193.04" y="88.9"/>
 <instance part="R2" gate="G$1" x="160.02" y="124.46" rot="MR90"/>
-<instance part="SUPPLY1" gate="G$1" x="111.76" y="111.76"/>
+<instance part="SUPPLY1" gate="G$1" x="104.14" y="111.76"/>
 <instance part="SUPPLY2" gate="G$1" x="27.94" y="170.18"/>
-<instance part="GND1" gate="1" x="60.96" y="132.08" rot="R180"/>
-<instance part="GND2" gate="1" x="60.96" y="114.3" rot="R180"/>
-<instance part="GND3" gate="1" x="106.68" y="132.08" rot="R180"/>
+<instance part="GND1" gate="1" x="73.66" y="129.54" rot="R180"/>
+<instance part="GND2" gate="1" x="73.66" y="114.3" rot="R180"/>
+<instance part="GND3" gate="1" x="129.54" y="134.62" rot="R180"/>
 <instance part="GND4" gate="1" x="20.32" y="149.86"/>
 <instance part="GND5" gate="1" x="27.94" y="149.86"/>
-<instance part="GND7" gate="1" x="104.14" y="114.3" rot="R180"/>
+<instance part="GND7" gate="1" x="114.3" y="114.3" rot="R180"/>
 <instance part="J1" gate="G$1" x="15.24" y="157.48"/>
-<instance part="C1" gate="G$1" x="27.94" y="157.48"/>
 <instance part="SUPPLY3" gate="G$1" x="160.02" y="132.08"/>
 <instance part="SUPPLY4" gate="G$1" x="167.64" y="132.08"/>
-<instance part="C2" gate="G$1" x="149.86" y="114.3" rot="R90"/>
 <instance part="GND6" gate="1" x="167.64" y="50.8"/>
 <instance part="JAVR" gate="G$1" x="81.28" y="162.56"/>
@@
 <instance part="SUPPLY7" gate="G$1" x="30.48" y="132.08"/>
 <instance part="JP2" gate="G$1" x="10.16" y="121.92"/>
+<instance part="C1" gate="G$1" x="27.94" y="157.48"/>
+<instance part="C2" gate="G$1" x="149.86" y="114.3" rot="R90"/>
 </instances>
 <busses>
@@
 <net name="GND" class="0">
 <segment>
-<pinref part="JPTIMER" gate="G$1" pin="2"/>
-<pinref part="GND1" gate="1" pin="GND"/>
-<wire x1="53.34" y1="127" x2="60.96" y2="127" width="0.1524" layer="91"/>
-<wire x1="60.96" y1="127" x2="60.96" y2="129.54" width="0.1524" layer="91"/>
-</segment>
-<segment>
-<pinref part="JPTOGGLE" gate="G$1" pin="2"/>
-<pinref part="GND2" gate="1" pin="GND"/>
-<wire x1="53.34" y1="109.22" x2="60.96" y2="109.22" width="0.1524" layer="91"/>
-<wire x1="60.96" y1="109.22" x2="60.96" y2="111.76" width="0.1524" layer="91"/>
-</segment>
-<segment>
-<pinref part="JPSPEAKER" gate="G$1" pin="2"/>
 <pinref part="GND3" gate="1" pin="GND"/>
-<wire x1="99.06" y1="127" x2="106.68" y2="127" width="0.1524" layer="91"/>
-<wire x1="106.68" y1="127" x2="106.68" y2="129.54" width="0.1524" layer="91"/>
+<pinref part="JPSPEAKER" gate="G$1" pin="1"/>
+<wire x1="99.06" y1="124.46" x2="129.54" y2="124.46" width="0.1524" layer="91"/>
+<wire x1="129.54" y1="124.46" x2="129.54" y2="132.08" width="0.1524" layer="91"/>
 </segment>
 <segment>
@@
 </segment>
 <segment>
-<pinref part="C1" gate="G$1" pin="2"/>
 <pinref part="GND5" gate="1" pin="GND"/>
 <wire x1="27.94" y1="154.94" x2="27.94" y2="152.4" width="0.1524" layer="91"/>
+<pinref part="C1" gate="G$1" pin="2"/>
 </segment>
 <segment>
@@
 </segment>
 <segment>
-<pinref part="JPDISPLAY" gate="G$1" pin="3"/>
-<wire x1="99.06" y1="109.22" x2="104.14" y2="109.22" width="0.1524" layer="91"/>
 <pinref part="GND7" gate="1" pin="GND"/>
-<wire x1="104.14" y1="111.76" x2="104.14" y2="109.22" width="0.1524" layer="91"/>
-</segment>
-</net>
-<net name="OUT_DISPLAY" class="0">
-<segment>
-<pinref part="JPDISPLAY" gate="G$1" pin="1"/>
-<wire x1="99.06" y1="104.14" x2="119.38" y2="104.14" width="0.1524" layer="91"/>
-<label x="114.3" y="104.14" size="1.778" layer="95"/>
-</segment>
-<segment>
-<pinref part="U1" gate="G$1" pin="PD6(AIN0)"/>
-<wire x1="218.44" y1="76.2" x2="226.06" y2="76.2" width="0.1524" layer="91"/>
-<label x="220.98" y="76.2" size="1.778" layer="95"/>
-</segment>
-</net>
-<net name="IN_TIMER" class="0">
+<wire x1="114.3" y1="111.76" x2="114.3" y2="106.68" width="0.1524" layer="91"/>
+<pinref part="JPDISPLAY" gate="G$1" pin="2"/>
+<wire x1="114.3" y1="106.68" x2="99.06" y2="106.68" width="0.1524" layer="91"/>
+</segment>
 <segment>
 <pinref part="JPTIMER" gate="G$1" pin="1"/>
 <wire x1="53.34" y1="124.46" x2="73.66" y2="124.46" width="0.1524" layer="91"/>
-<label x="68.58" y="124.46" size="1.778" layer="95"/>
-</segment>
+<pinref part="GND1" gate="1" pin="GND"/>
+<wire x1="73.66" y1="124.46" x2="73.66" y2="127" width="0.1524" layer="91"/>
+</segment>
+<segment>
+<pinref part="JPTOGGLE" gate="G$1" pin="1"/>
+<pinref part="GND2" gate="1" pin="GND"/>
+<wire x1="53.34" y1="106.68" x2="73.66" y2="106.68" width="0.1524" layer="91"/>
+<wire x1="73.66" y1="106.68" x2="73.66" y2="111.76" width="0.1524" layer="91"/>
+</segment>
+</net>
+<net name="IN_TIMER" class="0">
 <segment>
 <pinref part="U1" gate="G$1" pin="PD3(INT1)"/>
@@
 <label x="220.98" y="83.82" size="1.778" layer="95"/>
 </segment>
+<segment>
+<pinref part="JPTIMER" gate="G$1" pin="2"/>
+<wire x1="53.34" y1="127" x2="63.5" y2="127" width="0.1524" layer="91"/>
+<label x="58.42" y="127" size="1.778" layer="95"/>
+</segment>
 </net>
 <net name="IN_TOGGLE" class="0">
-<segment>
-<pinref part="JPTOGGLE" gate="G$1" pin="1"/>
-<wire x1="53.34" y1="106.68" x2="73.66" y2="106.68" width="0.1524" layer="91"/>
-<label x="68.58" y="106.68" size="1.778" layer="95"/>
-</segment>
 <segment>
 <pinref part="U1" gate="G$1" pin="PD2(INT0)"/>
@@
 <label x="220.98" y="86.36" size="1.778" layer="95"/>
 </segment>
-</net>
-<net name="N$1" class="0">
-<segment>
-<pinref part="JPSPEAKER" gate="G$1" pin="1"/>
-<pinref part="R1" gate="G$1" pin="1"/>
-<wire x1="99.06" y1="124.46" x2="101.6" y2="124.46" width="0.1524" layer="91"/>
+<segment>
+<pinref part="JPTOGGLE" gate="G$1" pin="2"/>
+<wire x1="53.34" y1="109.22" x2="63.5" y2="109.22" width="0.1524" layer="91"/>
+<label x="58.42" y="109.22" size="1.778" layer="95"/>
 </segment>
 </net>
@@
 <segment>
 <pinref part="R1" gate="G$1" pin="2"/>
-<wire x1="111.76" y1="124.46" x2="119.38" y2="124.46" width="0.1524" layer="91"/>
-<label x="114.3" y="124.46" size="1.778" layer="95"/>
+<wire x1="111.76" y1="127" x2="119.38" y2="127" width="0.1524" layer="91"/>
+<label x="111.76" y="127" size="1.778" layer="95"/>
 </segment>
 <segment>
@@
 <wire x1="17.78" y1="165.1" x2="27.94" y2="165.1" width="0.1524" layer="91"/>
 <wire x1="27.94" y1="165.1" x2="27.94" y2="170.18" width="0.1524" layer="91"/>
-<pinref part="C1" gate="G$1" pin="1"/>
 <wire x1="27.94" y1="165.1" x2="27.94" y2="162.56" width="0.1524" layer="91"/>
 <junction x="27.94" y="165.1"/>
+<pinref part="C1" gate="G$1" pin="1"/>
 </segment>
 <segment>
@@
 </segment>
 <segment>
-<pinref part="JPDISPLAY" gate="G$1" pin="2"/>
-<wire x1="99.06" y1="106.68" x2="111.76" y2="106.68" width="0.1524" layer="91"/>
 <pinref part="SUPPLY1" gate="G$1" pin="VCC"/>
-<wire x1="111.76" y1="111.76" x2="111.76" y2="106.68" width="0.1524" layer="91"/>
+<wire x1="104.14" y1="111.76" x2="104.14" y2="109.22" width="0.1524" layer="91"/>
+<pinref part="JPDISPLAY" gate="G$1" pin="3"/>
+<wire x1="104.14" y1="109.22" x2="99.06" y2="109.22" width="0.1524" layer="91"/>
 </segment>
 </net>
@@
 <wire x1="170.18" y1="114.3" x2="160.02" y2="114.3" width="0.1524" layer="91"/>
 <wire x1="160.02" y1="114.3" x2="160.02" y2="119.38" width="0.1524" layer="91"/>
-<pinref part="C2" gate="G$1" pin="2"/>
 <wire x1="160.02" y1="114.3" x2="152.4" y2="114.3" width="0.1524" layer="91"/>
 <junction x="160.02" y="114.3"/>
 <label x="162.56" y="114.3" size="1.778" layer="95"/>
+<pinref part="C2" gate="G$1" pin="2"/>
 </segment>
 </net>
@@
 <label x="220.98" y="88.9" size="1.778" layer="95"/>
 </segment>
+<segment>
+<pinref part="JPDISPLAY" gate="G$1" pin="1"/>
+<wire x1="99.06" y1="104.14" x2="119.38" y2="104.14" width="0.1524" layer="91"/>
+<label x="114.3" y="104.14" size="1.778" layer="95"/>
+</segment>
 </net>
 <net name="DTR" class="0">
@@
 </segment>
 <segment>
-<pinref part="C2" gate="G$1" pin="1"/>
 <wire x1="144.78" y1="114.3" x2="137.16" y2="114.3" width="0.1524" layer="91"/>
 <label x="137.16" y="114.3" size="1.778" layer="95"/>
+<pinref part="C2" gate="G$1" pin="1"/>
 </segment>
 </net>
@@
 </segment>
 </net>
+<net name="N$1" class="0">
+<segment>
+<pinref part="JPSPEAKER" gate="G$1" pin="2"/>
+<pinref part="R1" gate="G$1" pin="1"/>
+<wire x1="99.06" y1="127" x2="101.6" y2="127" width="0.1524" layer="91"/>
+</segment>
+</net>
